File: Etherwave-GateCV.kicad_pcb (KiCad board)
At the start: 2 copper layers, 67 x 60 mm, 80 parts, among them J1 Etherwave Brd, J2 Volume CV, J3 Pitch CV, J4 Gate, Q1 PMP4501Y, Q2 PMBT3906, Q3 PMP4501Y, U1 LM13700, U2 CD4093, U3 CD4093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

Commit message: added missing connection U7-A-1, C14, P1-1, R14. replaces hotfix
Connections:
- RV1 pad 1: Net-(RV1-Pad1) -> Net-(C14-Pad2)
- U7 pad 1: Net-(RV1-Pad1) -> Net-(C14-Pad2)
Routing:
- net Net-(C14-Pad2): track 3.82 -> 22.7 mm, vias 0 -> 1
- net Net-(RV1-Pad1): track 9.62 -> 0.00 mm
Other:
- board text added: "v1.1 2024.11"
- board text removed: "v1.0 2023.05"
